Commit message: prepare view_robot.launch file
* hide obsolete urdfs for now

File: fanuc_lrmate200id_support/urdf/lrmate200id7l.urdf.xacro (robot description, xacro)
@@ -2,4 +2,9 @@
 <robot name="fanuc_lrmate200id7l" xmlns:xacro="http://ros.org/wiki/xacro">
   <xacro:include filename="$(find fanuc_lrmate200id_support)/urdf/lrmate200id7l_macro.xacro"/>
-  <xacro:fanuc_lrmate200id7l prefix=""/>
+  <link name="world"/>
+  <xacro:fanuc_lrmate200id7l
+  prefix=""
+  parent="world">
+  <origin xyz="0 0 0" rpy="0 0 0"/>
+  </xacro:fanuc_lrmate200id7l>
 </robot>

File: fanuc_lrmate200id_support/urdf/lrmate200id7l_macro.xacro (robot description, xacro)
@@ -2,6 +2,6 @@
 <robot xmlns:xacro="http://ros.org/wiki/xacro">
   <xacro:include filename="$(find fanuc_resources)/urdf/common_materials.xacro"/>
-  <xacro:macro name="fanuc_lrmate200id7l" params="prefix">
-    <!-- links: main serial chain -->
+  <xacro:macro name="fanuc_lrmate200id7l" params="prefix parent *origin">
+    <!-- links - main serial chain -->
     <link name="${prefix}base_link">
       <visual>
@@ -109,5 +109,5 @@
       </collision>
     </link>
-    <!-- joints: main serial chain -->
+    <!-- joints - main serial chain -->
     <joint name="${prefix}joint_1" type="revolute">
       <origin xyz="0 0 0.330" rpy="0 0 0" />
@@ -152,5 +152,11 @@
       <limit effort="0" lower="${radians(-360)}" upper="${radians(360)}" velocity="${radians(1000)}" />
     </joint>
-    <!-- ROS-Industrial 'base' frame: base_link to Fanuc World Coordinates transform -->
+    <!-- parent_to_base_link fixes base_link to the environment -->
+    <joint name="${prefix}parent_to_base_link" type="fixed">
+      <xacro:insert_block name="origin" />
+      <parent link="${parent}" />
+      <child link="${prefix}base_link" />
+    </joint>
+    <!-- ROS-Industrial 'base' frame - base_link to Fanuc World Coordinates transform -->
     <link name="${prefix}base" />
     <joint name="${prefix}base_link-base" type="fixed">
@@ -159,5 +165,5 @@
       <child link="${prefix}base"/>
     </joint>
-    <!-- ROS-Industrial 'flange' frame: attachment point for EEF models -->
+    <!-- ROS-Industrial 'flange' frame - attachment point for EEF models -->
     <link name="${prefix}flange" />
     <joint name="${prefix}link_6-flange" type="fixed">
@@ -166,5 +172,5 @@
       <child link="${prefix}flange" />
     </joint>
-    <!-- ROS-Industrial 'tool0' frame: all-zeros tool frame -->
+    <!-- ROS-Industrial 'tool0' frame - all-zeros tool frame -->
     <link name="${prefix}tool0" />
     <joint name="${prefix}flange-tool0" type="fixed">
